File: eagle/flank_detection.brd (EAGLE design)
At the start: 160 x 100 mm, 10 parts, among them IC1 74AC04N, IC2 74AC14N, IC3 74AC86N

Commit message: Edited board
Parts:
- moved R1 40.5 mm to (12.1, 45.7), turned to 270 degrees
- moved C1 30.0 mm to (12.1, 38.1), turned to 270 degrees
- moved SV2 2.54 mm to (45.7, 22.9)
Routing:
- net GND: track 0.00 -> 141.9 mm
- net VCC: track 0.00 -> 72.0 mm
- net N$1: track 0.00 -> 36.4 mm, vias 0 -> 1
- net N$7: track 0.00 -> 35.9 mm, vias 0 -> 1
- net N$3: track 0.00 -> 28.1 mm
- net N$5: track 0.00 -> 25.2 mm
- net N$6: track 0.00 -> 18.6 mm
- net N$4: track 0.00 -> 17.6 mm
- net N$2: track 0.00 -> 11.8 mm
